Commit message: corrected axis to make i and comma , keys on the keyboard correspond to back and forward. Added Ros remapping to subscribe to cmd_vel

File: description/gazebo_control.xacro (robot description, xacro)
@@ -1,21 +1,25 @@
 <?xml version="1.0"?>
 <robot xmlns:xacro="http://www.ros.org/wiki/xacro"  >
-     <gazebo>
-        <plugin name='diff_drive' filename='libgazebo_ros_diff_drive.so'>
-         <!-- Wheel Information -->
-            <left_joint>left_wheel_joint</left_joint>
-            <right_joint>right_wheel_joint</right_joint>
-            <wheel_separation>0.254</wheel_separation>
-            <wheel_diameter>0.085</wheel_diameter>
-         <!-- Limits -->
-            <max_wheel_torque>200</max_wheel_torque>
-            <max_wheel_acceleration>10.0</max_wheel_acceleration>
-         <!-- Output -->
-            <odometry_frame>odom</odometry_frame>
-            <robot_base_frame>base_link</robot_base_frame>
-            <publish_odom>true</publish_odom>
-            <publish_odom_tf>true</publish_odom_tf>
-            <publish_wheel_tf>true</publish_wheel_tf>
-        </plugin>
-     </gazebo>
+  <gazebo>
+    <plugin name='diff_drive' filename='libgazebo_ros_diff_drive.so'>
+      <!-- ROS 2 remapping -->
+      <ros>
+        <remapping>cmd_vel:=/cmd_vel</remapping>
+      </ros>
+      <!-- Wheel Information -->
+      <left_joint>left_wheel_joint</left_joint>
+      <right_joint>right_wheel_joint</right_joint>
+      <wheel_separation>0.254</wheel_separation>
+      <wheel_diameter>0.085</wheel_diameter>
+      <!-- Limits -->
+      <max_wheel_torque>100</max_wheel_torque>
+      <max_wheel_acceleration>5.0</max_wheel_acceleration>
+      <!-- Output -->
+      <odometry_frame>odom</odometry_frame>
+      <robot_base_frame>base_link</robot_base_frame>
+      <publish_odom>true</publish_odom>
+      <publish_odom_tf>true</publish_odom_tf>
+      <publish_wheel_tf>true</publish_wheel_tf>
+    </plugin>
+  </gazebo>
 </robot>

File: description/robot_core.xacro (robot description, xacro)
@@ -73,5 +73,5 @@
         <child link="right_wheel"/>
         <origin xyz="0 -0.127 0" rpy="-${pi/2} 0 0"/>
-        <axis xyz="0 0 -1"/>
+        <axis xyz="0 0 1"/>
     </joint>
     <link name="right_wheel">
@@ -105,5 +105,5 @@
                 <sphere radius="0.0425" />
             </geometry>
-            <material name="black"/>
+            <material name="orange"/>
         </visual>
          <collision>
@@ -117,5 +117,5 @@
     </link>
       <gazebo reference="frontCaster_wheel">
-        <material>Gazebo/Black </material>
+        <material>Gazebo/Orange </material>
         <mu1 value="0.001"/>
         <mu2 value="0.001"/>
