Commit message: lidar fixed

File: description/lidar.xacro (robot description, xacro)
@@ -29,5 +29,5 @@
     <sensor name="laser" type="ray">
       <pose>0 0 0 0 0 0</pose>
-      <visualize>true</visualize>
+      <visualize>false</visualize>
       <update_rate>10</update_rate>
       <ray>

File: description/robot.urdf.xacro (robot description, xacro)
@@ -3,3 +3,5 @@
    <xacro:include filename="robot_core.xacro" />
    <xacro:include filename="gazebo_control.xacro"/>
+   <xacro:include filename="lidar.xacro"/>
+   <xacro:include filename="camera.xacro"/>
 </robot>

File: description/robot_core.xacro (robot description, xacro)
@@ -61,5 +61,5 @@
             <collision>
                 <geometry>
-                    <cylinder length="0.04" radius="0.0425" />
+                    <sphere radius="0.0425" />
                 </geometry>
             </collision>
@@ -87,5 +87,5 @@
         <collision>
             <geometry>
-                <cylinder length="0.04" radius="0.0425" />
+                <sphere radius="0.0425" />
             </geometry>
         </collision>
@@ -131,18 +131,18 @@
     </joint>
     <link name="backCaster_wheel">
-        <visual>
-            <geometry>
-                <sphere radius="0.0425" />
-            </geometry>
-            <material name="black"/>
-        </visual>
-        <collision>
-            <geometry>
-                <sphere radius="0.0425" />
-            </geometry>
-        </collision>
-        <xacro:inertial_sphere mass="0.1" radius="0.0425">
-            <origin xyz="0 0 0" rpy="0 0 0"/>
-        </xacro:inertial_sphere>
+<visual>
+    <geometry>
+        <sphere radius="0.0425" />
+    </geometry>
+    <material name="black"/>
+</visual>
+<collision>
+    <geometry>
+        <sphere radius="0.0425" />
+    </geometry>
+</collision>
+<xacro:inertial_sphere mass="0.1" radius="0.0425">
+    <origin xyz="0 0 0" rpy="0 0 0"/>
+</xacro:inertial_sphere>
     </link>
     <gazebo reference="backCaster_wheel">
