Commit message: added inertial file

File: description/robot_core.xacro (robot description, xacro)
@@ -28,4 +28,10 @@
             <material name="white"/>
         </visual>
+         <collision>
+            <origin xyz="0.105 0 0.05" rpy="0 0 0"/>
+            <geometry>
+                <cylinder radius="0.11" length="0.10" />
+            </geometry>
+        </collision>
     </link>
     <!-- LEFT WHEEL -->
@@ -33,5 +39,5 @@
         <parent link="base_link"/>
         <child link="left_wheel"/>
-        <origin xyz="0 0.135 0" rpy="-${pi/2} 0 0"/>
+        <origin xyz="0 0.127 0" rpy="-${pi/2} 0 0"/>
         <axis xyz="0 0 1"/>
         </joint>
@@ -43,4 +49,9 @@
             <material name="blue"/>
         </visual>
+        <collision>
+            <geometry>
+                <cylinder length="0.04" radius="0.0425" />
+            </geometry>
+        </collision>
         </link>
      <!-- RIGHT WHEEL -->
@@ -48,5 +59,5 @@
         <parent link="base_link"/>
         <child link="right_wheel"/>
-        <origin xyz="0 -0.135 0" rpy="-${pi/2} 0 0"/>
+        <origin xyz="0 -0.127 0" rpy="-${pi/2} 0 0"/>
         <axis xyz="0 0 -1"/>
     </joint>
@@ -58,4 +69,9 @@
         <material name="blue"/>
     </visual>
+    <collision>
+        <geometry>
+            <cylinder length="0.04" radius="0.0425" />
+        </geometry>
+    </collision>
     </link>
     <!-- FRONT CASTER WHEEL -->
@@ -63,5 +79,5 @@
         <parent link="chassis"/>
         <child link="frontCaster_wheel"/>
-        <origin xyz="0.21 0 0" rpy="0 0 0"/>
+        <origin xyz="0.21 0 -0.0425" rpy="0 0 0"/>
     </joint>
     <link name="frontCaster_wheel">
@@ -72,4 +88,9 @@
             <material name="black"/>
         </visual>
+         <collision>
+            <geometry>
+                <sphere radius="0.0425" />
+            </geometry>
+        </collision>
     </link>
      <!-- back CASTER WHEEL -->
@@ -77,5 +98,5 @@
         <parent link="chassis"/>
         <child link="backCaster_wheel"/>
-        <origin xyz="0 0 0" rpy="0 0 0"/>
+        <origin xyz="0 0 -0.0425" rpy="0 0 0"/>
     </joint>
     <link name="backCaster_wheel">
@@ -86,4 +107,9 @@
             <material name="black"/>
         </visual>
+        <collision>
+            <geometry>
+                <sphere radius="0.0425" />
+            </geometry>
+        </collision>
     </link>
 </robot>

Commit message: finished urdf contents

File: description/robot_core.xacro (robot description, xacro)
@@ -1,4 +1,5 @@
 <?xml version="1.0"?>
 <robot xmlns:xacro="http://www.ros.org/wiki/xacro" >
+    <xacro:include filename="inertial_macros.xacro"/>
     <material name="white">
         <color rgba="1 1 1 1"/>
@@ -24,5 +25,5 @@
             <origin xyz="0.105 0 0.05" rpy="0 0 0"/>
             <geometry>
-                <cylinder radius="0.11" length="0.10" />
+                <cylinder radius="0.105" length="0.10" />
             </geometry>
             <material name="white"/>
@@ -31,16 +32,42 @@
             <origin xyz="0.105 0 0.05" rpy="0 0 0"/>
             <geometry>
-                <cylinder radius="0.11" length="0.10" />
+                <cylinder radius="0.105" length="0.10" />
             </geometry>
         </collision>
+        <xacro:inertial_cylinder mass="0.8" length="0.1" radius="0.11">
+            <origin xyz="0 0 0" rpy="0 0 0"/>
+        </xacro:inertial_cylinder>
     </link>
     <!-- LEFT WHEEL -->
-        <joint name="left_wheel_joint" type="continuous">
+    <joint name="left_wheel_joint" type="continuous">
         <parent link="base_link"/>
         <child link="left_wheel"/>
         <origin xyz="0 0.127 0" rpy="-${pi/2} 0 0"/>
         <axis xyz="0 0 1"/>
-        </joint>
-        <link name="left_wheel">
+    </joint>
+    <link name="left_wheel">
+            <visual>
+                <geometry>
+                    <cylinder length="0.04" radius="0.0425" />
+                </geometry>
+                <material name="blue"/>
+            </visual>
+            <collision>
+                <geometry>
+                    <cylinder length="0.04" radius="0.0425" />
+                </geometry>
+            </collision>
+            <xacro:inertial_cylinder mass="0.1" length="0.04" radius="0.0425">
+            <origin xyz="0 0 0" rpy="0 0 0"/>
+            </xacro:inertial_cylinder>
+    </link>
+     <!-- RIGHT WHEEL -->
+    <joint name="right_wheel_joint" type="continuous">
+        <parent link="base_link"/>
+        <child link="right_wheel"/>
+        <origin xyz="0 -0.127 0" rpy="-${pi/2} 0 0"/>
+        <axis xyz="0 0 -1"/>
+    </joint>
+    <link name="right_wheel">
         <visual>
             <geometry>
@@ -54,24 +81,7 @@
             </geometry>
         </collision>
-        </link>
-     <!-- RIGHT WHEEL -->
-    <joint name="right_wheel_joint" type="continuous">
-        <parent link="base_link"/>
-        <child link="right_wheel"/>
-        <origin xyz="0 -0.127 0" rpy="-${pi/2} 0 0"/>
-        <axis xyz="0 0 -1"/>
-    </joint>
-    <link name="right_wheel">
-    <visual>
-        <geometry>
-            <cylinder length="0.04" radius="0.0425" />
-        </geometry>
-        <material name="blue"/>
-    </visual>
-    <collision>
-        <geometry>
-            <cylinder length="0.04" radius="0.0425" />
-        </geometry>
-    </collision>
+        <xacro:inertial_cylinder mass="0.1" length="0.04" radius="0.0425">
+            <origin xyz="0 0 0" rpy="0 0 0"/>
+        </xacro:inertial_cylinder>
     </link>
     <!-- FRONT CASTER WHEEL -->
@@ -79,5 +89,5 @@
         <parent link="chassis"/>
         <child link="frontCaster_wheel"/>
-        <origin xyz="0.21 0 -0.0425" rpy="0 0 0"/>
+        <origin xyz="0.19 0 -0.0425" rpy="0 0 0"/>
     </joint>
     <link name="frontCaster_wheel">
@@ -93,4 +103,7 @@
             </geometry>
         </collision>
+        <xacro:inertial_sphere mass="0.1" radius="0.0425">
+             <origin xyz="0 0 0" rpy="0 0 0"/>
+        </xacro:inertial_sphere>
     </link>
      <!-- back CASTER WHEEL -->
@@ -98,5 +111,5 @@
         <parent link="chassis"/>
         <child link="backCaster_wheel"/>
-        <origin xyz="0 0 -0.0425" rpy="0 0 0"/>
+        <origin xyz="0.02 0 -0.0425" rpy="0 0 0"/>
     </joint>
     <link name="backCaster_wheel">
@@ -112,4 +125,7 @@
             </geometry>
         </collision>
+        <xacro:inertial_sphere mass="0.1" radius="0.0425">
+            <origin xyz="0 0 0" rpy="0 0 0"/>
+        </xacro:inertial_sphere>
     </link>
 </robot>

Commit message: Added camera to the workspace

File: description/robot_core.xacro (robot description, xacro)
@@ -13,4 +13,7 @@
     <material name="black">
         <color rgba="0 0 0 1"/>
+    </material>
+    <material name="red">
+        <color rgba="1 0 0 1"/>
     </material>
     <link name="base_link">

Commit message: added Pi gemetry

File: description/robot_core.xacro (robot description, xacro)
@@ -49,5 +49,5 @@
         <parent link="base_link"/>
         <child link="left_wheel"/>
-        <origin xyz="0 0.127 0" rpy="-${pi/2} 0 0"/>
+        <origin xyz="0.09 0.127 0" rpy="-${pi/2} 0 0"/>
         <axis xyz="0 0 1"/>
     </joint>
@@ -61,5 +61,5 @@
             <collision>
                 <geometry>
-                    <sphere radius="0.0425" />
+                    <cylinder length="0.001" radius="0.0425" />
                 </geometry>
             </collision>
@@ -75,5 +75,5 @@
         <parent link="base_link"/>
         <child link="right_wheel"/>
-        <origin xyz="0 -0.127 0" rpy="-${pi/2} 0 0"/>
+        <origin xyz="0.09 -0.127 0" rpy="-${pi/2} 0 0"/>
         <axis xyz="0 0 1"/>
     </joint>
@@ -87,5 +87,5 @@
         <collision>
             <geometry>
-                <sphere radius="0.0425" />
+                    <cylinder length="0.001" radius="0.0425" />
             </geometry>
         </collision>
@@ -97,5 +97,5 @@
         <material>Gazebo/Blue </material>
     </gazebo>
-    <!-- FRONT CASTER WHEEL -->
+    <!-- FRONT CASTER WHEEL
     <joint name="frontCaster_wheel_joint" type="fixed">
         <parent link="chassis"/>
@@ -123,5 +123,5 @@
         <mu1 value="0.001"/>
         <mu2 value="0.001"/>
-    </gazebo>
+    </gazebo> -->
      <!-- back CASTER WHEEL -->
     <joint name="backCaster_wheel_joint" type="fixed">
@@ -151,3 +151,29 @@
         <mu2 value="0.001"/>
     </gazebo>
+      <!-- PI -->
+    <joint name="raspi_joint" type="fixed">
+         <parent link="chassis"/>
+         <child link="raspi_box"/>
+         <origin xyz="0.06 0.04 0" rpy="0 0 0"/>
+    </joint>
+    <link name="raspi_box">
+        <visual>
+            <geometry>
+                <box size="0.084 0.057 0.014"/>
+            </geometry>
+            <material name="blue"/>
+        </visual>
+        <collision>
+           <origin xyz="0.06 -0.04 0.12" rpy="0 0 0"/>
+           <geometry>
+                <box size="0.084 0.057 0.014"/>
+            </geometry>
+        </collision>
+        <xacro:inertial_box mass="0.1" x="0.084" y="0.057" z="0.014">
+            <origin xyz="0 0 0" rpy="0 0 0"/>
+        </xacro:inertial_box>
+    </link>
+    <gazebo reference="raspi_box">
+        <material>Gazebo/Black </material>
+    </gazebo>
 </robot>
