Commit message: Added 15 seconds delay time to spawning part of script to allow the publisher to completely load before spawning

File: description/robot.urdf.xacro (robot description, xacro)
@@ -2,3 +2,4 @@
 <robot xmlns:xacro="http://www.ros.org/wiki/xacro"  name="robot">
    <xacro:include filename="robot_core.xacro" />
+   <xacro:include filename="gazebo_control.xacro"/>
 </robot>

File: description/robot_core.xacro (robot description, xacro)
@@ -39,4 +39,7 @@
         </xacro:inertial_cylinder>
     </link>
+    <gazebo reference="chassis">
+        <material>Gazebo/white </material>
+    </gazebo>
     <!-- LEFT WHEEL -->
     <joint name="left_wheel_joint" type="continuous">
@@ -62,4 +65,7 @@
             </xacro:inertial_cylinder>
     </link>
+    <gazebo reference="left_wheel">
+        <material>Gazebo/Blue </material>
+    </gazebo>
      <!-- RIGHT WHEEL -->
     <joint name="right_wheel_joint" type="continuous">
@@ -85,4 +91,7 @@
         </xacro:inertial_cylinder>
     </link>
+    <gazebo reference="right_wheel">
+        <material>Gazebo/Blue </material>
+    </gazebo>
     <!-- FRONT CASTER WHEEL -->
     <joint name="frontCaster_wheel_joint" type="fixed">
@@ -107,4 +116,9 @@
         </xacro:inertial_sphere>
     </link>
+      <gazebo reference="frontCaster_wheel">
+        <material>Gazebo/Black </material>
+        <mu1 value="0.001"/>
+        <mu2 value="0.001"/>
+    </gazebo>
      <!-- back CASTER WHEEL -->
     <joint name="backCaster_wheel_joint" type="fixed">
@@ -129,3 +143,8 @@
         </xacro:inertial_sphere>
     </link>
+    <gazebo reference="backCaster_wheel">
+        <material>Gazebo/Black </material>
+        <mu1 value="0.001"/>
+        <mu2 value="0.001"/>
+    </gazebo>
 </robot>

Commit message: worked on paths

File: description/robot.urdf.xacro (robot description, xacro)
@@ -2,6 +2,7 @@
 <robot xmlns:xacro="http://www.ros.org/wiki/xacro"  name="robot">
    <xacro:include filename="robot_core.xacro" />
-   <xacro:include filename="gazebo_control.xacro"/>
+   <xacro:include filename="ros2_control.xacro"/>
+   <!-- <xacro:include filename="gazebo_control.xacro"/> -->
    <xacro:include filename="lidar.xacro"/>
-   <xacro:include filename="camera.xacro"/>
+   <!-- <xacro:include filename="camera.xacro"/> -->
 </robot>

File: description/robot_core.xacro (robot description, xacro)
@@ -43,5 +43,5 @@
     </link>
     <gazebo reference="chassis">
-        <material>Gazebo/white </material>
+        <material>Gazebo/White </material>
     </gazebo>
     <!-- LEFT WHEEL -->
@@ -155,5 +155,5 @@
          <parent link="chassis"/>
          <child link="raspi_box"/>
-         <origin xyz="0.06 0.04 0" rpy="0 0 0"/>
+         <origin xyz="0.06 0.04 0.1" rpy="0 0 0"/>
     </joint>
     <link name="raspi_box">
