Commit message: changed code configuration to work in gazebo fortress

File: description/camera.xacro (robot description, xacro)
@@ -1,5 +1,5 @@
 <?xml version="1.0"?>
 <robot xmlns:xacro="http://www.ros.org/wiki/xacro">
-  <!-- Joint: attach laser to chassis -->
+  <!-- Joint: attach camera to chassis -->
   <joint name="camera_joint" type="fixed">
     <parent link="chassis"/>
@@ -7,13 +7,14 @@
     <origin xyz="0.11 -0.04 0.12" rpy="0 0 0"/>
   </joint>
-  <!-- Laser link -->
+  <!-- Camera body link -->
   <link name="camera_link">
     <visual>
-        <geometry>
-            <box size="0.010 0.03 0.03"/>
-        </geometry>
-        <material name="red"/>
+      <geometry>
+        <box size="0.010 0.03 0.03"/>
+      </geometry>
+      <material name="red"/>
     </visual>
   </link>
+  <!-- Optical frame for camera -->
   <joint name="camera_optical_joint" type="fixed">
     <origin xyz="0 0 0" rpy="${-pi/2} 0 ${-pi/2}" />
@@ -21,28 +22,27 @@
     <child link="camera_link_optical" />
   </joint>
-  <link name="camera_link_optical"></link>
-    <!-- Gazebo sensor -->
-    <gazebo reference="camera_link">
-      <material>Gazebo/Red</material>
-      <sensor name="camera" type="camera">
-        <pose> 0 0 0 0 0 0 </pose>
-        <visualize>true</visualize>
-        <update_rate>10</update_rate>
-        <camera>
-            <horizontal_fov>1.089</horizontal_fov>
-            <image>
-              <format>R8G8B8</format>
-              <width>640</width>
-              <height>480</height>
-            </image>
-            <clip>
-              <near>0.05</near>
-              <far>8.0</far>
-            </clip>
-        </camera>
-          <plugin name="camera_controller" filename="libgazebo_ros_camera.so">
-            <frame_name>camera_link_optical</frame_name>
-          </plugin>
-      </sensor>
+  <link name="camera_link_optical" />
+  <!-- Gazebo/Ignition camera sensor -->
+  <gazebo reference="camera_link">
+    <material>Gazebo/Red</material>
+    <sensor name="camera" type="camera">
+      <pose>0 0 0 0 0 0</pose>
+      <visualize>true</visualize>
+      <update_rate>30</update_rate>
+      <camera>
+        <horizontal_fov>1.089</horizontal_fov>
+        <image>
+          <format>R8G8B8</format>
+          <width>640</width>
+          <height>480</height>
+        </image>
+        <clip>
+          <near>0.05</near>
+          <far>8.0</far>
+        </clip>
+      </camera>
+      <!-- In Ignition, no ROS plugin — topics will be published on /camera -->
+      <always_on>true</always_on>
+    </sensor>
   </gazebo>
 </robot>

File: description/lidar.xacro (robot description, xacro)
@@ -24,11 +24,10 @@
     </xacro:inertial_cylinder>
   </link>
-  <!-- Gazebo sensor -->
+  <!-- Ignition Gazebo LIDAR sensor -->
   <gazebo reference="laser_frame">
-    <material>Gazebo/Red</material>
-    <sensor name="laser" type="ray">
+    <sensor name="lidar" type="gpu_lidar">
       <pose>0 0 0 0 0 0</pose>
-      <visualize>false</visualize>
       <update_rate>10</update_rate>
+      <visualize>true</visualize>
       <ray>
         <scan>
@@ -46,13 +45,4 @@
         </range>
       </ray>
-      <!-- ROS 2 Gazebo plugin -->
-      <plugin name="gazebo_ros_laser" filename="libgazebo_ros_ray_sensor.so">
-        <ros>
-          <namespace>/</namespace>
-          <remapping>scan:=/scan</remapping>
-        </ros>
-        <output_type>sensor_msgs/msg/LaserScan</output_type>
-        <frame_name>laser_frame</frame_name>
-      </plugin>
     </sensor>
   </gazebo>

File: description/ros2_control.xacro (robot description, xacro)
@@ -1,8 +1,8 @@
 <?xml version="1.0"?>
 <robot xmlns:xacro="http://www.ros.org/wiki/xacro">
-  <!-- ros2_control setup -->
+  <!-- ros2_control configuration -->
   <ros2_control name="GazeboSystem" type="system">
     <hardware>
-      <plugin>gazebo_ros2_control/GazeboSystem</plugin>
+    <plugin>ros_gz_sim_ros2_control/GazeboSystem</plugin>
     </hardware>
     <joint name="left_wheel_joint">
@@ -23,9 +23,5 @@
     </joint>
   </ros2_control>
-  <!-- Gazebo plugin to load ros2_control -->
-  <gazebo>
-    <plugin name="gazebo_ros2_control" filename="libgazebo_ros2_control.so">
-      <parameters>$(find neural_knights)/config/my_controllers.yaml</parameters>
-    </plugin>
-  </gazebo>
+  <!-- 🔴 Remove Gazebo classic plugin block -->
+  <!-- In Fortress, ros2_control is started from your launch file using ros2_control_node -->
 </robot>
